File: PCB/Unibots_PCB.kicad_sch (KiCad schematic)
At the start: 21 parts, among them J1 Conn_01x04_Socket, J2 Conn_01x04_Socket, J3 Conn_01x04_Socket, J4 Conn_01x04_Socket, J5 Conn_01x08_Socket, U1 DRV8833PW, U2 DRV8833PW

Commit message: add readme to repo
Other:
- note added: "Encoders"
Changed lines of the file:
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@@
 	(text "5V Regulator"
 		(exclude_from_sim no)
-		(at 112.014 79.248 0)
+		(at 146.812 80.772 0)
 		(effects
 			(font
@@
 		(effects
 			(font
+				(size 1.27 1.27)
+			)
+		)
+	)
+	(text "Encoders"
+		(exclude_from_sim no)
+		(at 123.698 80.264 0)
+		(effects
+			(font

Commit message: change 1
Other:
- note added: "5V Regulator 1"
- note added: "5V Regulator 2"
- note added: "Servo motor"
- note removed: "5V Regulator"
- note removed: "Encoders"
Changed lines of the file:
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@@
 	(generator_version "9.0")
 	(paper "A4")
+	(text "Servo motor"
+		(exclude_from_sim no)
+		(at 84.836 121.92 0)
+		(effects
+			(font
+				(size 1.27 1.27)
+			)
+		)
+	)
 	(text "Potential Dividers"
 		(exclude_from_sim no)
@@
 		)
 	)
-	(text "5V Regulator"
+	(text "5V Regulator 1"
 		(exclude_from_sim no)
 		(at 146.812 80.772 0)
@@
 		)
 	)
-	(text "Encoders"
+	(text "5V Regulator 2\n"
 		(exclude_from_sim no)
-		(at 123.698 80.264 0)
+		(at 145.288 114.554 0)
 		(effects
 			(font

Commit message: add new components
Parts:
- removed C1: 100nF, symbol Device:C
- removed C2: C_Polarized, symbol Device:C_Polarized
- removed U1, U2: DRV8833PW, Package_SO:TSSOP-16_4.4x5mm_P0.65mm, symbol Driver_Motor:DRV8833PW
- added C1, C8: 10uF, symbol Device:C_Polarized
- added C10, C11: 10uF, Capacitor_SMD:C_1206_3216Metric_Pad1.33x1.80mm_HandSolder, symbol Device:C
- added C12: 10nF, Capacitor_SMD:C_0805_2012Metric_Pad1.18x1.45mm_HandSolder, symbol Device:C
- added C13, C2: 100nF, Capacitor_SMD:C_0805_2012Metric_Pad1.18x1.45mm_HandSolder, symbol Device:C
- added C14, C15: 47uF, Capacitor_SMD:C_1206_3216Metric_Pad1.33x1.80mm_HandSolder, symbol Device:C
- added C7: 100uF, symbol Device:C_Polarized
- added C9: 10uF, Capacitor_SMD:C_0805_2012Metric_Pad1.18x1.45mm_HandSolder, symbol Device:C
- added J10: Conn_02x19_Counter_Clockwise, Module:ESP32_DevkitC_V4, symbol Connector_Generic:Conn_02x19_Counter_Clockwise
- added J11, J12, J6, J7: Conn_01x03_Pin, Connector_PinSocket_2.54mm:PinSocket_1x03_P2.54mm_Vertical, symbol Connector:Conn_01x03_Pin
- added J13: Conn_01x08_Socket, Connector_PinHeader_2.54mm:PinHeader_1x08_P2.54mm_Vertical, symbol Connector:Conn_01x08_Socket
- added J8: Screw_Terminal_01x02, TerminalBlock:TerminalBlock_MaiXu_MX126-5.0-02P_1x02_P5.00mm, symbol Connector:Screw_Terminal_01x02
- added J9: Conn_02x20_Odd_Even, Connector_IDC:IDC-Header_2x20_P2.54mm_Vertical, symbol Connector_Generic:Conn_02x20_Odd_Even
- added JP1, JP2, JP3, JP4: SolderJumper_2_Open, Jumper:SolderJump_Big, symbol Jumper:SolderJumper_2_Open
- added L1: 6.8uH, Inductor_SMD:L_Coilcraft_XAL5020-XXX, symbol Device:L
- added Q1: PMOS, symbol Simulation_SPICE:PMOS
- added R10: 47k, Resistor_SMD:R_0805_2012Metric_Pad1.20x1.40mm_HandSolder, symbol Device:R
- added R11: 52.3k, Resistor_SMD:R_0805_2012Metric_Pad1.20x1.40mm_HandSolder, symbol Device:R
- added R12: 10k, Resistor_SMD:R_0805_2012Metric_Pad1.20x1.40mm_HandSolder, symbol Device:R
- added R13, R14, R9: 100k, Resistor_SMD:R_0805_2012Metric_Pad1.20x1.40mm_HandSolder, symbol Device:R
- added SW1: SW_SPST, symbol Switch:SW_SPST
- added U1, U3: TB6612FNG, Package_SO:SSOP-24_5.3x8.2mm_P0.65mm, symbol Driver_Motor:TB6612FNG
- added U4: AP64502, Package_SO:Diodes_SO-8EP, symbol Regulator_Switching:AP64502
- added U5: TLV76150DCY, Package_TO_SOT_SMD:SOT-223-3_TabPin2, symbol Regulator_Linear:TLV76150DCY
- C3, C6: value 2.2uF -> 100nF; footprint (none) -> Capacitor_SMD:C_0805_2012Metric_Pad1.18x1.45mm_HandSolder
- C4: footprint (none) -> Capacitor_SMD:C_0805_2012Metric_Pad1.18x1.45mm_HandSolder
- C5: value C_Polarized -> 10uF
- R1, R2, R3, R4, R5, R6, R7, R8: footprint (none) -> Resistor_SMD:R_0805_2012Metric_Pad1.20x1.40mm_HandSolder
Connections:
- net GND: now also C3.2, C4.2, C1.2, C10.1, C11.1, C12.1, C14.1, C15.1, C2.1, C7.2, C8.2, C9.1, J10.14 (Pin_14), J10.32 (Pin_32), J10.38 (Pin_38), J11.3 (Pin_3), J12.3 (Pin_3), J13.7 (Pin_7), J13.8 (Pin_8), J6.3 (Pin_3), J7.3 (Pin_3), J8.2 (Pin_2), J9.14 (Pin_14), J9.20 (Pin_20), J9.25 (Pin_25), J9.30 (Pin_30), J9.34 (Pin_34), J9.39 (Pin_39), J9.6 (Pin_6), J9.9 (Pin_9), R10.2, R12.2, R9.2, U1.10 (PGND2), U1.18 (GND), U1.3 (PGND1), U1.4 (PGND1), U1.9 (PGND2), U3.10 (PGND2), U3.18 (GND), U3.3 (PGND1), U3.4 (PGND1), U3.9 (PGND2), U4.7 (GND), U4.9 (PAD), U5.1 (GND); no longer C3.1, C4.1
- net INA: now also U3.21 (AIN1)
- net INB: now also U3.22 (AIN2)
- net INC: now also U3.17 (BIN1)
- net IND: now also U3.16 (BIN2)
- net INE: now also U1.21 (AIN1)
- net INF: now also U1.22 (AIN2)
- net ING: now also U1.17 (BIN1)
- net INH: now also U1.16 (BIN2)
- net MotorBackLeft+: now also U1.1 (AO1), U1.2 (AO1)
- net MotorBackLeft-: now also U1.5 (AO2), U1.6 (AO2)
- net MotorBackRight+: now also U1.11 (BO1), U1.12 (BO1)
- net MotorBackRight-: now also U1.7 (BO2), U1.8 (BO2)
- net MotorFrontLeft+: now also U3.1 (AO1), U3.2 (AO1)
- net MotorFrontLeft-: now also U3.5 (AO2), U3.6 (AO2)
- net MotorFrontRight+: now also U3.11 (BO1), U3.12 (BO1)
- net MotorFrontRight-: now also U3.7 (BO2), U3.8 (BO2)
- net V_motor1: now reaches C5.1
- net V_motor1: now also C6.2, JP3.1 (A), JP4.1 (A), U3.13 (VM2), U3.14 (VM3), U3.24 (VM1); no longer C4.2
- net 5V renamed 5V_PI
- net 5V_PI: now also C14.2, C15.2, J13.3 (Pin_3), J13.4 (Pin_4), J6.2 (Pin_2), J7.2 (Pin_2), J9.2 (Pin_2), J9.4 (Pin_4), L1.2, R11.1; no longer J5.1 (Pin_1)
- new net: C13.1, L1.1, U4.8 (SW)
- new net: C13.2, U4.1 (BST)
- new net: R11.2, R12.1, U4.5 (FB)
- new net: Q1.2 (G), R9.1
- new net: C10.2, C11.2, U4.2 (VIN)
- new net: Q1.3 (S), SW1.1 (A)
- new net: R10.1, U4.4 (RT/CLK)
- new net: C12.2, U4.6 (SS)
- new net 3V3_ESP32: J10.1 (Pin_1)
- new net 3V3_PI: J9.1 (Pin_1), R13.1, R14.1
- new net 5V_LDO: C3.1, C4.1, C7.1, J10.19 (Pin_19), J13.1 (Pin_1), J13.2 (Pin_2), J5.1 (Pin_1), U1.19 (STBY), U1.20 (VCC), U3.19 (STBY), U3.20 (VCC), U5.2 (VO)
- new net 5V_motor: JP2.2 (B), JP4.2 (B)
- new net Bat+: C9.2, J8.1 (Pin_1), Q1.1 (D)
- new net COM: J11.1 (Pin_1), R13.2
- new net COM2: J12.1 (Pin_1), R14.2
- new net ENA: U3.23 (PWMA)
- new net ENB: U3.15 (PWMB)
- new net ENC: U1.23 (PWMA)
- new net END: U1.15 (PWMB)
- new net NC: J11.2 (Pin_2)
- new net NC2: J12.2 (Pin_2)
- new net Servo1_Sig: J6.1 (Pin_1)
- new net Servo2_Sig: J7.1 (Pin_1)
- new net V_motor2: C1.1, C2.2, JP1.1 (A), JP2.1 (A), U1.13 (VM2), U1.14 (VM3), U1.24 (VM1)
- new net Vin: C8.1, JP1.2 (B), JP3.2 (B), SW1.2 (B), U5.3 (VI)
Other:
- note added: "Additional Pinout (In case)"
- note added: "Connected to COM when not pressed"
- note added: "Connected to GPIO Pin. HIGH when not pressed, LOW when pressed"
- note added: "ESP32 Pinout"
- note added: "Limit Switches"
- note added: "Make sure VGS threshold is above 12V (~20V)"
- note added: "Motor Supply Selection"
- note added: "NO:Connected to COM when pressed"
- note added: "Potential Dividers for Ultrasonic Sensors"
- note added: "Raspberry Pi Pinout"
- note added: "Reverse Polarity Protection"
- note added: "Tantalum cap"
- note removed: "Potential Dividers"
- moved on the sheet: R1, R2, R3, R4, R5, R6, R7, R8

Commit message: Most schematic layout
Parts:
- removed Q1: PMOS, symbol Simulation_SPICE:PMOS
- added C16, C17: 10uF, Capacitor_SMD:C_1206_3216Metric_Pad1.33x1.80mm_HandSolder, symbol Device:C
- added C18: 100nF, Capacitor_SMD:C_0805_2012Metric_Pad1.18x1.45mm_HandSolder, symbol Device:C
- added C19: 10nF, Capacitor_SMD:C_0805_2012Metric_Pad1.18x1.45mm_HandSolder, symbol Device:C
- added C20, C21: 47uF, Capacitor_SMD:C_1206_3216Metric_Pad1.33x1.80mm_HandSolder, symbol Device:C
- added J14, J15, J16, J17: Screw_Terminal_01x02, TerminalBlock:TerminalBlock_MaiXu_MX126-5.0-02P_1x02_P5.00mm, symbol Connector:Screw_Terminal_01x02
- added L2: 6.8uH, Inductor_SMD:L_Coilcraft_XAL5020-XXX, symbol Device:L
- added Q2: Q_PMOS_GDS, Package_TO_SOT_SMD:TO-252-3_TabPin2, symbol Transistor_FET:Q_PMOS_GDS
- added R15: 47k, Resistor_SMD:R_0805_2012Metric_Pad1.20x1.40mm_HandSolder, symbol Device:R
- added R16: 77.5k, Resistor_SMD:R_0805_2012Metric_Pad1.20x1.40mm_HandSolder, symbol Device:R
- added R17: 10k, Resistor_SMD:R_0805_2012Metric_Pad1.20x1.40mm_HandSolder, symbol Device:R
- added R18, R19: 330Ω, Resistor_SMD:R_0805_2012Metric_Pad1.20x1.40mm_HandSolder, symbol Device:R
- added SW2: SW_SPDT, symbol Switch:SW_SPDT
- added U2: AP64502, Package_SO:Diodes_SO-8EP, symbol Regulator_Switching:AP64502
- C1, C5: footprint (none) -> Capacitor_Tantalum_SMD:CP_EIA-3216-10_Kemet-I_HandSolder
- C7: footprint (none) -> Capacitor_Tantalum_SMD:CP_EIA-7343-15_Kemet-W_HandSolder
- C8: footprint (none) -> Capacitor_SMD:C_1206_3216Metric_Pad1.33x1.80mm_HandSolder
Connections:
- net SCL is gone; now on net SCL_ESP32: J5.3 (Pin_3)
- net SDA is gone; now on net SDA_ESP32: J5.4 (Pin_4)
- net 3V3_PI: now also J9.17 (Pin_17)
- net Bat+: now also Q2.2 (D)
- net COM: now also J9.31 (Pin_31)
- net COM2: now also J9.16 (Pin_16)
- net ENA: now also J10.7 (Pin_7)
- net ENB: now also J10.8 (Pin_8)
- net ENC: now also J10.15 (Pin_15)
- net END: now also J10.37 (Pin_37)
- net Echo1Pi: now also J9.19 (Pin_19)
- net Echo2Pi: now also J9.21 (Pin_21)
- net Echo3Pi: now also J9.23 (Pin_23)
- net Echo4Pi: now also J9.29 (Pin_29)
- net GND: now also J13.5 (Pin_5), J13.6 (Pin_6), C16.1, C17.1, C19.1, C20.1, C21.1, R15.2, R17.2, SW2.3 (C), U2.7 (GND), U2.9 (PAD)
- net INA: now also J10.9 (Pin_9)
- net INB: now also J10.10 (Pin_10)
- net INC: now also J10.11 (Pin_11)
- net IND: now also J10.12 (Pin_12)
- net INE: now also J10.31 (Pin_31)
- net INF: now also J10.30 (Pin_30)
- net ING: now also J10.26 (Pin_26)
- net INH: now also J10.24 (Pin_24)
- net MotorBackLeft+: now also J15.1 (Pin_1)
- net MotorBackLeft-: now also J15.2 (Pin_2)
- net MotorBackRight+: now also J17.1 (Pin_1)
- net MotorBackRight-: now also J17.2 (Pin_2)
- net MotorFrontLeft+: now also J14.1 (Pin_1)
- net MotorFrontLeft-: now also J14.2 (Pin_2)
- net MotorFrontRight+: now also J16.1 (Pin_1)
- net MotorFrontRight-: now also J16.2 (Pin_2)
- net Servo1_Sig: now also J9.33 (Pin_33)
- net Servo2_Sig: now also J9.32 (Pin_32)
- net Trig1: now also J9.7 (Pin_7)
- net Trig2: now also J9.11 (Pin_11)
- net Trig3: now also J9.13 (Pin_13)
- net Trig4: now also J9.15 (Pin_15)
- net Vin: now also C10.2, C11.2, U4.2 (VIN), C16.2, C17.2, SW2.1 (A), U2.2 (VIN), U2.3 (EN)
- net at R9.1: now also Q2.1 (G)
- net at SW1.1 (A): now also Q2.3 (S)
- net at U4.3 (EN): now also SW2.2 (B)
- net GPIO_16: now reaches J10.27 (Pin_27)
- net GPIO_16: now also R19.2
- net GPIO_17: now reaches J10.28 (Pin_28)
- net GPIO_17: now also R18.1
- net SDA_ESP32: now reaches J10.33 (Pin_33)
- net RX0: now reaches J10.34 (Pin_34)
- net TX0: now reaches J10.35 (Pin_35)
- net SCL_ESP32: now reaches J10.36 (Pin_36)
- net RXD_PI: now reaches J9.10 (Pin_10)
- net RXD_PI: now also R18.2
- net EXTRA_PI_GPIO1: now reaches J9.18 (Pin_18)
- net EXTRA_PI_GPIO2: now reaches J9.22 (Pin_22)
- net EXTRA_PI_GPIO3: now reaches J9.24 (Pin_24)
- net EXTRA_PI_GPIO4: now reaches J9.26 (Pin_26)
- net SDA_PI: now reaches J9.3 (Pin_3)
- net EXTRA_PI_GPIO5: now reaches J9.36 (Pin_36)
- net SCL_PI: now reaches J9.5 (Pin_5)
- net TXD_PI: now reaches J9.8 (Pin_8)
- net TXD_PI: now also R19.1
- net 5V_motor renamed 7V_motor
- net 7V_motor: now also C20.2, C21.2, L2.2, R16.1
- new net: R15.1, U2.4 (RT/CLK)
- new net: R16.2, R17.1, U2.5 (FB)
- new net: C18.1, L2.1, U2.8 (SW)
- new net: C18.2, U2.1 (BST)
- new net: C19.2, U2.6 (SS)
- no-connect marks 0 -> 13
Other:
- note added: "7V Regulator"
- note added: "Additional Power Pinout (In case)"
- note added: "Capacitors tantalum: 10uF - T491A106M016AT (https://uk.farnell.com/kemet/t491a106m016at/cap-10-f-16v-20-1206-smd/dp/1650980) 100uF - https://uk.farnell.com/avx/tajd107k020rnj/cap-100-f-20v-10-2917-smd/dp/1135058 PMOS - https://uk.farnell.com/rohm/rd3p01battl1/mosfet-p-ch-100v-10a-to-252/dp/4168776"
- note added: "Motor Terminals"
- note removed: "Additional Pinout (In case)"
- moved on the sheet: C7, C8, C9, J10, J13, J8, R9, SW1, U5

Commit message: change
Parts:
- removed C7: 100uF, Capacitor_Tantalum_SMD:CP_EIA-7343-15_Kemet-W_HandSolder, symbol Device:C_Polarized
- removed C8: 10uF, Capacitor_SMD:C_1206_3216Metric_Pad1.33x1.80mm_HandSolder, symbol Device:C_Polarized
- added C7, C8: 10uF, Capacitor_SMD:C_0805_2012Metric_Pad1.18x1.45mm_HandSolder, symbol Device:C
- C10, C11: footprint Capacitor_SMD:C_1206_3216Metric_Pad1.33x1.80mm_HandSolder -> Capacitor_SMD:C_0805_2012Metric_Pad1.18x1.45mm_HandSolder
Connections:
- net 5V_LDO: now also C7.2
- net GND: now also C7.1, C8.1
- net Vin: now also C8.2
Changed lines of the file:
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@@
 	)
 	(junction
+		(at 120.65 132.08)
+		(diameter 0)
+		(color 0 0 0 0)
+	)
+	(junction
 		(at 116.84 191.77)
 		(diameter 0)
@@
 		(color 0 0 0 0)
 	)
-	(junction
-		(at 120.65 132.08)
-		(diameter 0)
-		(color 0 0 0 0)
-	)
 	(no_connect
 		(at 227.33 132.08)
@@
 	(wire
 		(pts
-			(xy 118.11 132.08) (xy 120.65 132.08)
-		)
-		(stroke
-			(width 0)
-			(type default)
-		)
-	)
-	(wire
-		(pts
 			(xy 204.47 97.79) (xy 204.47 102.87)
 		)
@@
 	(wire
 		(pts
-			(xy 120.65 132.08) (xy 123.19 132.08)
+			(xy 118.11 132.08) (xy 120.65 132.08)
 		)
 		(stroke
@@
 	(wire
 		(pts
+			(xy 120.65 132.08) (xy 123.19 132.08)
+		)
+		(stroke
+			(width 0)
+			(type default)
+		)
+	)
+	(wire
+		(pts
 			(xy 128.27 171.45) (xy 132.08 171.45)
 		)
@@
 	)
 	(symbol
-		(lib_id "Device:C_Polarized")
-		(at 120.65 135.89 0)
-		(unit 1)
-		(exclude_from_sim no)
-		(in_bom yes)
-		(on_board yes)
-		(dnp no)
-		(property "Reference" "C8"
-			(at 116.84 135.89 0)
-			(effects
-				(font
-					(size 1.27 1.27)
-				)
-			)
-		)
-		(property "Value" "10uF"
-			(at 116.078 138.938 0)
-			(effects
-				(font
-					(size 1.27 1.27)
-				)
-			)
-		)
-		(property "Footprint" "Capacitor_SMD:C_1206_3216Metric_Pad1.33x1.80mm_HandSolder"
-			(at 121.6152 139.7 0)
-			(effects
-				(font
-					(size 1.27 1.27)
-				)
-				(hide yes)
-			)
-		)
-		(property "Datasheet" "~"
-			(at 120.65 135.89 0)
-			(effects
-				(font
-					(size 1.27 1.27)
-				)
-				(hide yes)
-			)
-		)
-		(property "Description" "Polarized capacitor"
-			(at 120.65 135.89 0)
-			(effects
-				(font
-					(size 1.27 1.27)
-				)
-				(hide yes)
-			)
-		)
-		(pin "2"
-		)
-		(pin "1"
-		)
-		(instances
-			(project "Unibots_PCB"
-				(path "/a1de844a-84f5-403a-bc32-d5187da60c13"
-					(reference "C8")
-					(unit 1)
-				)
-			)
-		)
-	)
-	(symbol
 		(lib_id "Connector:Screw_Terminal_01x02")
 		(at 205.74 26.67 0)
@@
 	(symbol
 		(lib_id "Device:C")
+		(at 120.65 135.89 180)
+		(unit 1)
+		(exclude_from_sim no)
+		(in_bom yes)
+		(on_board yes)
+		(dnp no)
+		(property "Reference" "C8"
+			(at 114.808 135.128 0)
+			(effects
+				(font
+					(size 1.27 1.27)
+				)
+				(justify right)
+			)
+		)
+		(property "Value" "10uF"
+			(at 114.046 139.192 0)
+			(effects
+				(font
+					(size 1.27 1.27)
+				)
+				(justify right)
+			)
+		)
+		(property "Footprint" "Capacitor_SMD:C_0805_2012Metric_Pad1.18x1.45mm_HandSolder"
+			(at 119.6848 132.08 0)
+			(effects
+				(font
+					(size 1.27 1.27)
+				)
+				(hide yes)
+			)
+		)
+		(property "Datasheet" "~"
+			(at 120.65 135.89 0)
+			(effects
+				(font
+					(size 1.27 1.27)
+				)
+				(hide yes)
+			)
+		)
+		(property "Description" "Unpolarized capacitor"
+			(at 120.65 135.89 0)
+			(effects
+				(font
+					(size 1.27 1.27)
+				)
+				(hide yes)
+			)
+		)
+		(pin "1"
+		)
+		(pin "2"
+		)
+		(instances
+			(project "Unibots_PCB"
+				(path "/a1de844a-84f5-403a-bc32-d5187da60c13"
+					(reference "C8")
+					(unit 1)
+				)
+			)
+		)
+	)
+	(symbol
+		(lib_id "Device:C")
 		(at 120.65 91.44 180)
 		(unit 1)
@@
 			)
 		)
-		(property "Footprint" "Capacitor_SMD:C_1206_3216Metric_Pad1.33x1.80mm_HandSolder"
+		(property "Footprint" "Capacitor_SMD:C_0805_2012Metric_Pad1.18x1.45mm_HandSolder"
 			(at 119.6848 87.63 0)
 			(effects
@@
 			)
 		)
-		(property "Footprint" "Capacitor_SMD:C_1206_3216Metric_Pad1.33x1.80mm_HandSolder"
+		(property "Footprint" "Capacitor_SMD:C_0805_2012Metric_Pad1.18x1.45mm_HandSolder"
 			(at 109.5248 86.36 0)
 			(effects
@@
 	)
 	(symbol
-		(lib_id "Device:C_Polarized")
-		(at 142.24 137.16 0)
-		(unit 1)
-		(exclude_from_sim no)
-		(in_bom yes)
-		(on_board yes)
-		(dnp no)
-		(property "Reference" "C7"
-			(at 138.43 137.16 0)
-			(effects
-				(font
-					(size 1.27 1.27)
-				)
-			)
-		)
-		(property "Value" "100uF"
-			(at 148.59 137.16 0)
-			(effects
-				(font
-					(size 1.27 1.27)
-				)
-			)
-		)
-		(property "Footprint" "Capacitor_Tantalum_SMD:CP_EIA-7343-15_Kemet-W_HandSolder"
-			(at 143.2052 140.97 0)
-			(effects
-				(font
-					(size 1.27 1.27)
-				)
-				(hide yes)
-			)
-		)
-		(property "Datasheet" "~"
-			(at 142.24 137.16 0)
-			(effects
-				(font
-					(size 1.27 1.27)
-				)
-				(hide yes)
-			)
-		)
-		(property "Description" "Polarized capacitor"
-			(at 142.24 137.16 0)
-			(effects
-				(font
-					(size 1.27 1.27)
-				)
-				(hide yes)
-			)
-		)
-		(pin "2"
-		)
-		(pin "1"
-		)
-		(instances
-			(project "Unibots_PCB"
-				(path "/a1de844a-84f5-403a-bc32-d5187da60c13"
-					(reference "C7")
-					(unit 1)
-				)
-			)
-		)
-	)
-	(symbol
 		(lib_id "Jumper:SolderJumper_2_Open")
 		(at 135.89 60.96 0)
@@
 					(unit 1)
 				)
+			)
+		)
+	)
+	(symbol
+		(lib_id "Device:C")
+		(at 142.24 137.16 180)
+		(unit 1)
+		(exclude_from_sim no)
+		(in_bom yes)
+		(on_board yes)
+		(dnp no)
+		(property "Reference" "C7"
+			(at 143.002 134.62 0)
+			(effects
+				(font
+					(size 1.27 1.27)
+				)
+				(justify right)
+			)
+		)
+		(property "Value" "10uF"
+			(at 145.796 137.414 0)
+			(effects
+				(font
+					(size 1.27 1.27)
+				)
+				(justify right)
+			)
+		)
+		(property "Footprint" "Capacitor_SMD:C_0805_2012Metric_Pad1.18x1.45mm_HandSolder"
+			(at 141.2748 133.35 0)
+			(effects
+				(font
+					(size 1.27 1.27)
+				)
+				(hide yes)
+			)
+		)
+		(property "Datasheet" "~"
+			(at 142.24 137.16 0)
+			(effects
+				(font
+					(size 1.27 1.27)
+				)
+				(hide yes)
+			)
+		)
+		(property "Description" "Unpolarized capacitor"
+			(at 142.24 137.16 0)
+			(effects
+				(font
+					(size 1.27 1.27)
+				)
+				(hide yes)
+			)
+		)
+		(pin "1"
+		)
+		(pin "2"
+		)
+		(instances
+			(project "Unibots_PCB"
+				(path "/a1de844a-84f5-403a-bc32-d5187da60c13"
+					(reference "C7")
+					(unit 1)
+				)

Commit message: pcb update
Parts:
- removed SW2: SW_SPDT, symbol Switch:SW_SPDT
- added C22, C23, C24, C25: 47uF, Capacitor_SMD:C_1206_3216Metric_Pad1.33x1.80mm_HandSolder, symbol Device:C
Connections:
- net 5V_PI: now also C22.2, C23.2
- net 7V_motor: now also C24.2, C25.2
- net GND: now also C22.1, C23.1, C24.1, C25.1
- net Vin: now also U4.3 (EN)
Other:
- moved on the sheet: C10, C11, C20, C21

Commit message: pcb design update
Parts:
- removed JP1, JP2, JP3, JP4: SolderJumper_2_Open, Jumper:SolderJump_Big, symbol Jumper:SolderJumper_2_Open
- removed SW1: SW_SPST, symbol Switch:SW_SPST
- added J18: Screw_Terminal_01x02, TerminalBlock:TerminalBlock_MaiXu_MX126-5.0-02P_1x02_P5.00mm, symbol Connector:Screw_Terminal_01x02
Connections:
- net V_motor1 is gone; now on net 7V_motor: C5.1, C6.2, U3.13 (VM2), U3.14 (VM3), U3.24 (VM1)
- net V_motor2 is gone; now on net 7V_motor: C1.1, C2.2, U1.13 (VM2), U1.14 (VM3), U1.24 (VM1)
- net MotorBackLeft+: now also U3.11 (BO1), U3.12 (BO1); no longer U1.1 (AO1), U1.2 (AO1)
- net MotorBackLeft-: now also U3.7 (BO2), U3.8 (BO2); no longer U1.5 (AO2), U1.6 (AO2)
- net MotorFrontRight+: now also U1.1 (AO1), U1.2 (AO1); no longer U3.11 (BO1), U3.12 (BO1)
- net MotorFrontRight-: now also U1.5 (AO2), U1.6 (AO2); no longer U3.7 (BO2), U3.8 (BO2)
- net Vin: now also J18.1 (Pin_1)
- net at Q2.3 (S): now also J18.2 (Pin_2)
Other:
- note added: "Switch"
- note removed: "Motor Supply Selection"

Commit message: pcb update
Parts:
- removed C1, C5: 10uF, Capacitor_Tantalum_SMD:CP_EIA-3216-10_Kemet-I_HandSolder, symbol Device:C_Polarized
- removed C16, C17: 10uF, Capacitor_SMD:C_1206_3216Metric_Pad1.33x1.80mm_HandSolder, symbol Device:C
- removed C18: 100nF, Capacitor_SMD:C_0805_2012Metric_Pad1.18x1.45mm_HandSolder, symbol Device:C
- removed C19: 10nF, Capacitor_SMD:C_0805_2012Metric_Pad1.18x1.45mm_HandSolder, symbol Device:C
- removed C20, C21, C24, C25: 47uF, Capacitor_SMD:C_1206_3216Metric_Pad1.33x1.80mm_HandSolder, symbol Device:C
- removed J13: Conn_01x08_Socket, Connector_PinHeader_2.54mm:PinHeader_1x08_P2.54mm_Vertical, symbol Connector:Conn_01x08_Socket
- removed L2: 6.8uH, Inductor_SMD:L_Coilcraft_XAL5020-XXX, symbol Device:L
- removed R17: 10k, Resistor_SMD:R_0805_2012Metric_Pad1.20x1.40mm_HandSolder, symbol Device:R
- removed U2: AP64502, Package_SO:Diodes_SO-8EP, symbol Regulator_Switching:AP64502
- added C1, C5: 10uF, Capacitor_SMD:C_0805_2012Metric_Pad1.18x1.45mm_HandSolder, symbol Device:C
- R15: value 47k -> 10k
- R16: value 77.5k -> 3.3k
Connections:
- net EXTRA_PI_GPIO3 is gone; now on net EXTRA_PI_GPIO5: J9.24 (Pin_24)
- net COM: now also J9.33 (Pin_33); no longer J9.31 (Pin_31)
- net COM2: now also J9.31 (Pin_31); no longer J9.16 (Pin_16)
- net ENA: now also J10.12 (Pin_12); no longer J10.7 (Pin_7)
- net ENB: now also J10.7 (Pin_7); no longer J10.8 (Pin_8)
- net ENC: now also J10.24 (Pin_24); no longer J10.15 (Pin_15)
- net END: now also J10.15 (Pin_15); no longer J10.37 (Pin_37)
- net EXTRA_PI_GPIO2: now also J9.32 (Pin_32); no longer J9.22 (Pin_22)
- net EXTRA_PI_GPIO5: no longer J9.36 (Pin_36)
- net Echo1Pi: now also J9.29 (Pin_29); no longer J9.19 (Pin_19)
- net Echo2Pi: now also J9.23 (Pin_23); no longer J9.21 (Pin_21)
- net Echo3Pi: now also J9.7 (Pin_7); no longer J9.23 (Pin_23)
- net Echo4Pi: now also J9.11 (Pin_11); no longer J9.29 (Pin_29)
- net GND: now also R16.1, C1.1, C5.1; no longer R15.2
- net INA: now also J10.10 (Pin_10); no longer J10.9 (Pin_9)
- net INB: now also J10.11 (Pin_11); no longer J10.10 (Pin_10)
- net INC: now also J10.9 (Pin_9); no longer J10.11 (Pin_11)
- net IND: now also J10.8 (Pin_8); no longer J10.12 (Pin_12)
- net INE: now also J10.30 (Pin_30); no longer J10.31 (Pin_31)
- net INF: now also J10.26 (Pin_26); no longer J10.30 (Pin_30)
- net ING: now also J10.31 (Pin_31); no longer J10.26 (Pin_26)
- net INH: now also J10.37 (Pin_37); no longer J10.24 (Pin_24)
- net Servo1_Sig: now also J9.35 (Pin_35); no longer J9.33 (Pin_33)
- net Servo2_Sig: now also J9.37 (Pin_37); no longer J9.32 (Pin_32)
- net Trig1: now also J9.19 (Pin_19); no longer J9.7 (Pin_7)
- net Trig2: now also J9.21 (Pin_21); no longer J9.11 (Pin_11)
- net Vin: now also C2.2, C6.2, R15.2, U1.13 (VM2), U1.14 (VM3), U1.24 (VM1), U3.13 (VM2), U3.14 (VM3), U3.24 (VM1), C1.2, C5.2
- net V_bat_measure: now reaches R15.1
- net V_bat_measure: now also J10.3 (Pin_3), R16.2
- removed net 7V_motor: C2.2, C6.2, R16.1, U1.13 (VM2), U1.14 (VM3), U1.24 (VM1), U3.13 (VM2), U3.14 (VM3), U3.24 (VM1)
- net EXTRA_PI_GPIO1: no longer names the net of J9.18 (Pin_18)
Other:
- note removed: "7V Regulator"
