File: PCB/Unibots_PCB.kicad_sch (KiCad schematic)
At the start: 58 parts, among them J1 Conn_01x04_Socket, J10 Conn_02x19_Counter_Clockwise, J11 Conn_01x03_Pin, J12 Conn_01x03_Pin, J14 Screw_Terminal_01x02, J15 Screw_Terminal_01x02, J16 Screw_Terminal_01x02, J17 Screw_Terminal_01x02, J18 Screw_Terminal_01x02, J2 Conn_01x04_Socket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

Commit message: update
Parts:
- Q2: value Q_PMOS_GDS -> RD3P01BATTL1
Changed lines of the file:
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@@
 			)
 		)
-		(property "Value" "Q_PMOS_GDS"
+		(property "Value" "RD3P01BATTL1"
 			(at 170.18 45.72 90)
 			(effects

Commit message: update
Parts:
- added JP1: SolderJumper_2_Open, Jumper:SolderJumper-2_P1.3mm_Open_TrianglePad1.0x1.5mm, symbol Jumper:SolderJumper_2_Open
Connections:
- net 5V_LDO: now also JP1.1 (A)
- net 5V_PI: now also JP1.2 (B)
Changed lines of the file:
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@@
 	)
 	(rectangle
-		(start 113.03 116.84)
-		(end 157.48 153.67)
+		(start 110.49 116.84)
+		(end 154.94 153.67)
 		(stroke
 			(width 0)
@@
 		)
 	)
+	(label "5V_LDO"
+		(at 167.64 134.62 180)
+		(effects
+			(font
+				(size 1.27 1.27)
+			)
+			(justify right bottom)
+		)
+	)
 	(label "TX0"
 		(at 240.03 99.06 0)
@@
 		)
 	)
+	(label "5V_PI"
+		(at 175.26 134.62 0)
+		(effects
+			(font
+				(size 1.27 1.27)
+			)
+			(justify left bottom)
+		)
+	)
 	(label "Vin"
 		(at 127 85.09 0)
@@
 					(unit 1)
 				)
+			)
+		)
+	)
+	(symbol
+		(lib_id "Jumper:SolderJumper_2_Open")
+		(at 171.45 134.62 0)
+		(unit 1)
+		(exclude_from_sim no)
+		(in_bom no)
+		(on_board yes)
+		(dnp no)
+		(fields_autoplaced yes)
+		(property "Reference" "JP1"
+			(at 171.45 128.27 0)
+			(effects
+				(font
+					(size 1.27 1.27)
+				)
+			)
+		)
+		(property "Value" "SolderJumper_2_Open"
+			(at 171.45 130.81 0)
+			(effects
+				(font
+					(size 1.27 1.27)
+				)
+			)
+		)
+		(property "Footprint" "Jumper:SolderJumper-2_P1.3mm_Open_TrianglePad1.0x1.5mm"
+			(at 171.45 134.62 0)
+			(effects
+				(font
+					(size 1.27 1.27)
+				)
+				(hide yes)
+			)
+		)
+		(property "Datasheet" "~"
+			(at 171.45 134.62 0)
+			(effects
+				(font
+					(size 1.27 1.27)
+				)
+				(hide yes)
+			)
+		)
+		(property "Description" "Solder Jumper, 2-pole, open"
+			(at 171.45 134.62 0)
+			(effects
+				(font
+					(size 1.27 1.27)
+				)
+				(hide yes)
+			)
+		)
+		(pin "1"
+		)
+		(pin "2"
+		)
+		(instances
+			(project ""
+				(path "/a1de844a-84f5-403a-bc32-d5187da60c13"
+					(reference "JP1")
+					(unit 1)
+				)
