File: PCB/Unibots_PCB.kicad_pcb (KiCad board)
At the start: 2 copper layers, 59.5 x 64.6 mm, 69 parts, among them J1 Conn_01x04_Socket, J10 Conn_02x19_Counter_Clockwise, J11 Conn_01x03_Pin, J12 Conn_01x03_Pin, J13 Conn_01x08_Socket, J14 Screw_Terminal_01x02, J15 Screw_Terminal_01x02, J16 Screw_Terminal_01x02, J17 Screw_Terminal_01x02, J2 Conn_01x04_Socket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

Commit message: pcb update
Parts:
- removed C7: 100uF, Capacitor_Tantalum_SMD:CP_EIA-7343-15_Kemet-W_HandSolder
- added C22: 47uF, Capacitor_SMD:C_1206_3216Metric_Pad1.33x1.80mm_HandSolder, F.Cu at (235.1, 91.4)
- added C23: 47uF, Capacitor_SMD:C_1206_3216Metric_Pad1.33x1.80mm_HandSolder, F.Cu at (235.1, 94.1)
- added C24: 47uF, Capacitor_SMD:C_1206_3216Metric_Pad1.33x1.80mm_HandSolder, F.Cu at (236.1, 115.5)
- added C25: 47uF, Capacitor_SMD:C_1206_3216Metric_Pad1.33x1.80mm_HandSolder, F.Cu at (236.1, 118.8)
- C10, C11, C8: footprint Capacitor_SMD:C_1206_3216Metric_Pad1.33x1.80mm_HandSolder -> Capacitor_SMD:C_0805_2012Metric_Pad1.18x1.45mm_HandSolder
- moved JP2 148.9 mm to (270.4, 100.2), turned to -90 degrees
- moved JP1 145.9 mm to (267.2, 100.2), turned to -90 degrees
- moved U5 134.5 mm to (224.6, 131.6)
- moved JP4 133.5 mm to (254.9, 99.8), turned to -90 degrees
- moved JP3 130.2 mm to (251.7, 99.9), turned to -90 degrees
- moved C9 128.7 mm to (252.0, 132.2), turned to 90 degrees
- moved C2 127.4 mm to (263.1, 100.8)
- moved C3 125.4 mm to (267.1, 90.7), turned to 90 degrees
- moved R9 122.8 mm to (255.7, 125.8)
- moved L2 121.5 mm to (232.0, 110.5)
- moved Q2 120.7 mm to (260.2, 130.8)
- moved C8 116.9 mm to (218.1, 132.4), turned to -90 degrees
- moved C4 111.5 mm to (253.3, 90.7), turned to 90 degrees
- moved U1 111.4 mm to (260.8, 92.4)
- moved C6 109.0 mm to (247.1, 100.9)
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Connections:
- C8 pad 1: /Vin -> GND
- C8 pad 2: GND -> /Vin
- U4 pad 3: unconnected-(U4-EN-Pad3) -> /Vin
Other:
- board size 59.5 x 64.6 mm -> 59.5 x 86.6 mm
- board text added: "5V Regulator"
- board text added: "7V Regulator"
- board text added: "Limit Switches"
- board text added: "MPU6050"
- board text added: "Motor Drivers"
- board text added: "Reverse Polarity Protection"
- board text added: "Servo Motors"
- board text added: "Ultrasonic Sensors"

Commit message: pcb design update
Parts:
- removed JP1, JP2, JP3, JP4: SolderJumper_2_Open, Jumper:SolderJump_Big
- added C7: 10uF, Capacitor_SMD:C_0805_2012Metric_Pad1.18x1.45mm_HandSolder, F.Cu at (235.5, 125.2)
- added J18: Screw_Terminal_01x02, TerminalBlock:TerminalBlock_MaiXu_MX126-5.0-02P_1x02_P5.00mm, F.Cu at (247.1, 131.1)
- moved J10 131.3 mm to (254.6, 62.3), turned to -90 degrees
- moved J1 91.1 mm to (268.9, 84.4), turned to -90 degrees
- moved J2 87.5 mm to (269.0, 79.7), turned to -90 degrees
- moved J6 85.5 mm to (264.0, 66.2), turned to 90 degrees
- moved J3 84.0 mm to (268.9, 75.2), turned to -90 degrees
- moved J4 80.9 mm to (268.9, 70.9), turned to -90 degrees
- moved J7 80.2 mm to (264.0, 62.2), turned to 90 degrees
- moved R1 77.3 mm to (253.7, 84.6), turned to -90 degrees
- moved R2 75.3 mm to (251.3, 84.6), turned to 90 degrees
- moved J5 74.5 mm to (236.3, 92.8), turned to -90 degrees
- moved R3 73.3 mm to (253.7, 80.2), turned to -90 degrees
- moved R4 71.5 mm to (251.3, 80.2), turned to 90 degrees
- moved R5 70.1 mm to (253.7, 75.6), turned to -90 degrees
- moved R6 68.7 mm to (251.3, 75.6), turned to 90 degrees
- moved R7 67.4 mm to (253.7, 71.2), turned to -90 degrees
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Connections:
- C1 pad 1: /V_motor2 -> /7V_motor
- C2 pad 2: /V_motor2 -> /7V_motor
- C5 pad 1: /V_motor1 -> /7V_motor
- C6 pad 2: /V_motor1 -> /7V_motor
- U1 pad 1: /MotorBackLeft+ -> /MotorFrontRight+
- U1 pad 13: /V_motor2 -> /7V_motor
- U1 pad 14: /V_motor2 -> /7V_motor
- U1 pad 2: /MotorBackLeft+ -> /MotorFrontRight+
- U1 pad 24: /V_motor2 -> /7V_motor
- U1 pad 5: /MotorBackLeft- -> /MotorFrontRight-
- U1 pad 6: /MotorBackLeft- -> /MotorFrontRight-
- U3 pad 11: /MotorFrontRight+ -> /MotorBackLeft+
- U3 pad 12: /MotorFrontRight+ -> /MotorBackLeft+
- U3 pad 13: /V_motor1 -> /7V_motor
- U3 pad 14: /V_motor1 -> /7V_motor
- U3 pad 24: /V_motor1 -> /7V_motor
- U3 pad 7: /MotorFrontRight- -> /MotorBackLeft-
- U3 pad 8: /MotorFrontRight- -> /MotorBackLeft-
Routing:
- net /5V_PI: track 0.00 -> 22.2 mm
- net /MotorBackRight+: track 0.00 -> 21.9 mm
- net /MotorFrontLeft+: track 0.00 -> 16.5 mm
- net /MotorBackRight-: track 0.00 -> 16.5 mm
- net /MotorFrontRight-: track 0.00 -> 16.4 mm
- net /MotorFrontLeft-: track 0.00 -> 12.7 mm
- net /MotorFrontRight+: track 0.00 -> 12.4 mm
- net /Echo1: track 0.00 -> 11.2 mm
- net /Echo4: track 0.00 -> 11.2 mm
- net /Echo2: track 0.00 -> 11.1 mm
- net /Echo3: track 0.00 -> 11.0 mm
- net /7V_motor: track 0.00 -> 8.74 mm
- net /MotorBackLeft-: track 0.00 -> 7.06 mm
- net /MotorBackLeft+: track 0.00 -> 6.35 mm
- net /5V_LDO: track 0.00 -> 6.30 mm
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- added copper zone on F.Cu, net /5V_LDO
- added copper zone on F.Cu, net /5V_PI
- added copper zone on F.Cu, net /7V_motor
- added copper zone on B.Cu, net /Bat+
- added copper zone on F.Cu, net /Bat+
- added copper zone on F.Cu, net /MotorBackLeft+
- added copper zone on F.Cu, net /MotorBackLeft-
- added copper zone on F.Cu, net /MotorBackRight+
- added copper zone on F.Cu, net /MotorBackRight-
- added copper zone on F.Cu, net /MotorFrontLeft+
- added copper zone on F.Cu, net /MotorFrontLeft-
- added copper zone on F.Cu, net /MotorFrontRight+
- added copper zone on F.Cu, net /MotorFrontRight-
- added copper zone on B.Cu, net /Vin
- added copper zone on F.Cu, net /Vin
- added copper zone on B.Cu, net Net-(J18-Pin_2)
- added copper zone on F.Cu, net Net-(J18-Pin_2)
- added copper zone on F.Cu, net Net-(U2-FB)
- added copper zone on F.Cu, net Net-(U2-SW)
- added copper zone on F.Cu, net Net-(U4-FB)
- added copper zone on F.Cu, net Net-(U4-SW)
Other:
- board size 59.5 x 86.6 mm -> 66 x 89 mm

Commit message: pcb update
Parts:
- removed C16, C17: 10uF, Capacitor_SMD:C_1206_3216Metric_Pad1.33x1.80mm_HandSolder
- removed C18: 100nF, Capacitor_SMD:C_0805_2012Metric_Pad1.18x1.45mm_HandSolder
- removed C19: 10nF, Capacitor_SMD:C_0805_2012Metric_Pad1.18x1.45mm_HandSolder
- removed C20, C21, C24, C25: 47uF, Capacitor_SMD:C_1206_3216Metric_Pad1.33x1.80mm_HandSolder
- removed J13: Conn_01x08_Socket, Connector_PinHeader_2.54mm:PinHeader_1x08_P2.54mm_Vertical
- removed L2: 6.8uH, Inductor_SMD:L_Coilcraft_XAL5020-XXX
- removed R17: 10k, Resistor_SMD:R_0805_2012Metric_Pad1.20x1.40mm_HandSolder
- removed U2: AP64502, Package_SO:Diodes_SO-8EP
- C1, C5: footprint Capacitor_Tantalum_SMD:CP_EIA-3216-10_Kemet-I_HandSolder -> Capacitor_SMD:C_0805_2012Metric_Pad1.18x1.45mm_HandSolder
- R15: value 47k -> 10k
- R16: value 77.5k -> 3.3k
- moved J18 75.2 mm to (212.5, 64.3), turned to -90 degrees
- moved C9 74.4 mm to (211.0, 86.5), turned to 0 degrees
- moved J8 71.3 mm to (212.8, 81.6), turned to 90 degrees
- moved C10 61.6 mm to (228.5, 62.4), turned to 180 degrees
- moved C11 59.1 mm to (227.5, 69.2), turned to 90 degrees
- moved Q2 59.0 mm to (221.5, 80.6), turned to -90 degrees
- moved R9 58.2 mm to (222.8, 72.6), turned to 180 degrees
- moved R10 54.2 mm to (231.0, 71.6), turned to 0 degrees
- moved U4 51.5 mm to (233.3, 67.1), turned to 0 degrees
- moved C13 50.7 mm to (234.8, 63.0), turned to 180 degrees
- moved R12 48.6 mm to (234.9, 71.6), turned to 180 degrees
- moved J17 45.9 mm to (235.0, 139.5), turned to 180 degrees
- moved C12 43.4 mm to (239.0, 67.7), turned to 180 degrees
- moved L1 43.3 mm to (240.5, 62.4), turned to 0 degrees
- moved R11 40.0 mm to (241.0, 71.5), turned to 180 degrees
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Connections:
- C1 pad 1: /7V_motor -> GND
- C1 pad 2: GND -> /Vin
- C2 pad 2: /7V_motor -> /Vin
- C5 pad 1: /7V_motor -> GND
- C5 pad 2: GND -> /Vin
- C6 pad 2: /7V_motor -> /Vin
- J10 pad 10: /INB -> /INA
- J10 pad 11: /INC -> /INB
- J10 pad 12: /IND -> /ENA
- J10 pad 15: /ENC -> /END
- J10 pad 24: /INH -> /ENC
- J10 pad 26: /ING -> /INF
- J10 pad 3: unconnected-(J10-Pin_3-Pad3) -> /V_bat_measure
- J10 pad 30: /INF -> /INE
- J10 pad 31: /INE -> /ING
- J10 pad 37: /END -> /INH
- J10 pad 7: /ENA -> /ENB
- J10 pad 8: /ENB -> /IND
- J10 pad 9: /INA -> /INC
- J9 pad 11: /Trig2 -> /Echo4Pi
- J9 pad 16: /COM2 -> unconnected-(J9-Pin_16-Pad16)
- J9 pad 18: /EXTRA_PI_GPIO1 -> unconnected-(J9-Pin_18-Pad18)
- J9 pad 19: /Echo1Pi -> /Trig1
- J9 pad 21: /Echo2Pi -> /Trig2
- J9 pad 22: /EXTRA_PI_GPIO2 -> unconnected-(J9-Pin_22-Pad22)
- J9 pad 23: /Echo3Pi -> /Echo2Pi
- J9 pad 24: /EXTRA_PI_GPIO3 -> /EXTRA_PI_GPIO5
- J9 pad 29: /Echo4Pi -> /Echo1Pi
- J9 pad 31: /COM -> /COM2
- J9 pad 32: /Servo2_Sig -> /EXTRA_PI_GPIO2
- J9 pad 33: /Servo1_Sig -> /COM
- J9 pad 35: unconnected-(J9-Pin_35-Pad35) -> /Servo1_Sig
- J9 pad 36: /EXTRA_PI_GPIO5 -> unconnected-(J9-Pin_36-Pad36)
- J9 pad 37: unconnected-(J9-Pin_37-Pad37) -> /Servo2_Sig
- J9 pad 7: /Trig1 -> /Echo3Pi
- R15 pad 1: Net-(U2-RT/CLK) -> /V_bat_measure
- R15 pad 2: GND -> /Vin
- R16 pad 1: /7V_motor -> GND
- R16 pad 2: Net-(U2-FB) -> /V_bat_measure
- U1 pad 13: /7V_motor -> /Vin
- U1 pad 14: /7V_motor -> /Vin
- U1 pad 24: /7V_motor -> /Vin
- U3 pad 13: /7V_motor -> /Vin
- U3 pad 14: /7V_motor -> /Vin
- U3 pad 24: /7V_motor -> /Vin
Routing:
- net /Vin: track 0.00 -> 121.7 mm, vias 10 -> 2
- net /5V_LDO: track 6.30 -> 107.7 mm, vias 0 -> 3
- net /RXD_PI: track 0.00 -> 72.6 mm, vias 0 -> 1
- net /GPIO_16: track 0.00 -> 60.6 mm, vias 0 -> 4
- net /3V3_PI: track 0.00 -> 58.8 mm
- net /END: track 0.00 -> 52.1 mm, vias 0 -> 1
- net /5V_PI: track 22.2 -> 71.1 mm
- net /IND: track 0.00 -> 48.4 mm, vias 0 -> 1
- net /ENB: track 0.00 -> 47.6 mm, vias 0 -> 1
- net /INC: track 0.00 -> 47.4 mm, vias 0 -> 1
- net /ENA: track 0.00 -> 45.1 mm, vias 0 -> 1
- net /INB: track 0.00 -> 44.5 mm, vias 0 -> 1
- net /INA: track 0.00 -> 44.4 mm, vias 0 -> 1
- net /Echo2Pi: track 2.40 -> 44.4 mm, vias 0 -> 1
- net /Trig2: track 0.00 -> 38.5 mm
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- added copper zone on B.Cu, net GND
- added copper zone on F.Cu, net GND
- removed copper zone on F.Cu, net /7V_motor
- removed copper zone on B.Cu, net /Vin
- removed copper zone on F.Cu, net Net-(U2-FB)
- removed copper zone on F.Cu, net Net-(U2-SW)
Other:
- board size 66 x 89 mm -> 58 x 96.8 mm
- board text removed: "7V Regulator"
- board text removed: "Limit Switches"
- board text removed: "Reverse Polarity Protection"

Commit message: update
Routing:
- net /5V_PI: track 71.1 -> 72.2 mm
Other:
- board text removed: "Servo Motors"
- board text removed: "Ultrasonic Sensors"
Changed lines of the file:
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@@
 			(plot_on_all_layers_selection 0x00000000_00000000_00000000_00000000)
 			(disableapertmacros no)
-			(usegerberextensions no)
+			(usegerberextensions yes)
 			(usegerberattributes yes)
 			(usegerberadvancedattributes yes)
-			(creategerberjobfile yes)
+			(creategerberjobfile no)
 			(dashed_line_dash_ratio 12.000000)
 			(dashed_line_gap_ratio 3.000000)
@@
 			(outputformat 1)
 			(mirror no)
-			(drillshape 1)
+			(drillshape 0)
 			(scaleselection 1)
-			(outputdirectory "")
+			(outputdirectory "Output")
 		)
 	)
@@
 		(tags "Through hole socket strip THT 1x03 2.54mm single row")
 		(property "Reference" "J6"
-			(at 4.15 -2.96 90)
+			(at -0.215 -2.795 90)
 			(layer "F.SilkS")
 			(effects
@@
 		(tags "Through hole socket strip THT 1x03 2.54mm single row")
 		(property "Reference" "J7"
-			(at -4.245 -3.625 90)
+			(at 0.14 -2.61 90)
 			(layer "F.SilkS")
 			(effects
@@
 		)
 	)
-	(gr_text "Servo Motors"
-		(at 273.275 55.035 0)
-		(layer "F.SilkS")
-		(effects
-			(font
-				(size 0.8 0.8)
-				(thickness 0.1)
-				(bold yes)
-			)
-			(justify left bottom)
-		)
-	)
-	(gr_text "Ultrasonic Sensors\n"
-		(at 249.89 78.93 0)
-		(layer "F.SilkS")
-		(effects
-			(font
-				(size 0.8 0.8)
-				(thickness 0.1)
-				(bold yes)
-			)
-			(justify left bottom)
-		)
-	)
 	(gr_text "MPU6050"
 		(at 234.02 98.485526 0)
@@
 	)
 	(segment
-		(start 242.96 81.72)
-		(end 242.96 73.03)
+		(start 208.9 51.35)
+		(end 208.25 52)
 		(width 2)
 		(layer "F.Cu")
@@
 	)
 	(segment
-		(start 242.96 73.03)
-		(end 243.86 72.13)
+		(start 208.25 55.42)
+		(end 210.54 57.71)
+		(width 2)
+		(layer "F.Cu")
+		(net 8)
+	)
+	(segment
+		(start 242.96 81.72)
+		(end 242.96 73.03)
 		(width 2)
 		(layer "F.Cu")
@@
 	)
 	(segment
-		(start 209 52.211)
-		(end 209 56.17)
+		(start 242.96 73.03)
+		(end 243.86 72.13)
 		(width 2)
 		(layer "F.Cu")
@@
 	)
 	(segment
-		(start 211.24 51.35)
-		(end 209.861 51.35)
+		(start 210.54 57.71)
+		(end 241.25 57.71)
 		(width 2)
 		(layer "F.Cu")
@@
 	)
 	(segment
-		(start 241.25 57.71)
-		(end 243.32 59.78)
+		(start 211.24 51.35)
+		(end 208.9 51.35)
 		(width 2)
 		(layer "F.Cu")
@@
 	)
 	(segment
-		(start 209.861 51.35)
-		(end 209 52.211)
+		(start 208.25 52)
+		(end 208.25 55.42)
 		(width 2)
 		(layer "F.Cu")
@@
 	)
 	(segment
-		(start 209 56.17)
-		(end 210.54 57.71)
+		(start 241.25 57.71)
+		(end 243.32 59.78)
 		(width 2)
 		(layer "F.Cu")
@@
 	)
 	(segment
-		(start 210.54 57.71)
-		(end 241.25 57.71)
-		(width 2)
-		(layer "F.Cu")
-		(net 8)
-	)
-	(segment
 		(start 224.8 103.95)
 		(end 222.74 103.95)
@@
 	)
 	(segment
-		(start 254.02 123.855526)
-		(end 254.02 111.945526)
+		(start 254.25 123.625526)
+		(end 254.25 110.145526)
 		(width 0.25)
 		(layer "B.Cu")
@@
 	)
 	(segment
-		(start 236.48 92.375526)
-		(end 235.46 92.375526)
-		(width 0.25)
-		(layer "B.Cu")
-		(net 50)
-	)
-	(segment
-		(start 235.25 92.155526)
-		(end 235.25 90.635526)
+		(start 251.43 126.445526)
+		(end 254.25 123.625526)
 		(width 0.25)
 		(layer "B.Cu")
@@
 	)
 	(segment
-		(start 251.43 126.445526)
-		(end 254.02 123.855526)
+		(start 236.48 92.375526)
+		(end 235.46 92.375526)
 		(width 0.25)
 		(layer "B.Cu")
@@
 	)
 	(segment
-		(start 254.02 111.945526)
-		(end 254.02 109.915526)
+		(start 235.25 92.155526)
+		(end 235.25 90.635526)
 		(width 0.25)
 		(layer "B.Cu")
@@
 	)
 	(segment
-		(start 235.46 92.365526)
-		(end 235.25 92.155526)
+		(start 254.25 110.145526)
+		(end 251.54 107.435526)
 		(width 0.25)
 		(layer "B.Cu")
@@
 	)
 	(segment
-		(start 254.02 109.915526)
-		(end 251.54 107.435526)
+		(start 235.46 92.365526)
+		(end 235.25 92.155526)
 		(width 0.25)
 		(layer "B.Cu")

Commit message: update
Parts:
- moved C22 0.22 mm to (246.5, 61.5)
Routing:
- net /ENB: track 47.6 -> 48.5 mm
- net /ENA: track 45.1 -> 44.3 mm
- net /INC: track 47.6 -> 47.0 mm
- net /IND: track 48.4 -> 47.8 mm
- net GND: vias 8 -> 70
Other:
- board text removed: "5V Regulator"
- board text removed: "MPU6050"
- board text removed: "Motor Drivers"

Commit message: update
Parts:
- added G***: LOGO, Logos:logo_medium2, F.Cu at (210.6, 137.9)
- added JP1: SolderJumper_2_Open, Jumper:SolderJumper-2_P1.3mm_Open_TrianglePad1.0x1.5mm, F.Cu at (241.8, 95.5)
- Q2: value Q_PMOS_GDS -> RD3P01BATTL1
Routing:
- net /5V_LDO: track 107.7 -> 131.5 mm, vias 3 -> 5
- net /Vin: track 121.7 -> 134.3 mm, vias 2 -> 6
- net /5V_PI: track 72.2 -> 81.8 mm
- net /V_bat_measure: track 33.2 -> 35.1 mm
- net GND: vias 70 -> 71
